File: split56/split56.sch (KiCad schematic (older format))
At the start: 42 parts, among them J1 AudioJack4, J2 AudioJack4, J3 AudioJack4, J4 AudioJack4, SW1 SW_DIP_x02, SW10 SW_Push, SW11 SW_Push, SW12 SW_Push, SW13 SW_Push, SW14 SW_Push, SW15 SW_Push, SW16 SW_Push, SW17 SW_Push, SW18 SW_Push, SW19 SW_Push, SW2 SW_Push, SW20 SW_Push, SW21 SW_Push, SW22 SW_Push, SW23 SW_Push, SW24 SW_Push, SW25 SW_Push, SW26 SW_Push, SW27 SW_Push, SW28 SW_Push, SW29 SW_Push, SW3 SW_Push, SW4 SW_Push, SW5 SW_Push, SW6 SW_Push, SW7 SW_Push, SW8 SW_Push, SW9 SW_Push, U1 TCA9555PWR, U2 TCA9555PWR

Commit message: Design main circuit
Connections:
- net GND: no longer J2.S, J4.S
- net VCC: no longer J2.T, J4.T
- no-connect marks 6 -> 10
Changed lines of the file:
@@
 EESchema Schematic File Version 4
+LIBS:split56-cache
 EELAYER 26 0
 EELAYER END
@@
 	1    0    0    -1
 $EndComp
-$Comp
-L power:GND #PWR05
-U 1 1 5CAE13D9
-P 3000 1950
-F 0 "#PWR05" H 3000 1700 50  0001 C CNN
-F 1 "GND" V 3005 1822 50  0000 R CNN
-F 2 "" H 3000 1950 50  0001 C CNN
-F 3 "" H 3000 1950 50  0001 C CNN
-	1    3000 1950
-	0    -1   -1   0
-$EndComp
-$Comp
-L power:VCC #PWR06
-U 1 1 5CAE13DF
-P 3000 2250
-F 0 "#PWR06" H 3000 2100 50  0001 C CNN
-F 1 "VCC" V 3017 2378 50  0000 L CNN
-F 2 "" H 3000 2250 50  0001 C CNN
-F 3 "" H 3000 2250 50  0001 C CNN
-	1    3000 2250
-	0    1    1    0
-$EndComp
 Text GLabel 3000 2150 2    50   Input ~ 0
 INT
@@
 	1    2800 2950
 	1    0    0    -1
-$EndComp
-$Comp
-L power:GND #PWR011
-U 1 1 5CAE13EE
-P 3000 2850
-F 0 "#PWR011" H 3000 2600 50  0001 C CNN
-F 1 "GND" V 3005 2722 50  0000 R CNN
-F 2 "" H 3000 2850 50  0001 C CNN
-F 3 "" H 3000 2850 50  0001 C CNN
-	1    3000 2850
-	0    -1   -1   0
-$EndComp
-$Comp
-L power:VCC #PWR012
-U 1 1 5CAE13F4
-P 3000 3150
-F 0 "#PWR012" H 3000 3000 50  0001 C CNN
-F 1 "VCC" V 3017 3278 50  0000 L CNN
-F 2 "" H 3000 3150 50  0001 C CNN
-F 3 "" H 3000 3150 50  0001 C CNN
-	1    3000 3150
-	0    1    1    0
 $EndComp
 Text GLabel 3000 3050 2    50   Input ~ 0
@@
 Text GLabel 10800 3750 3    50   Input ~ 0
 R4C7
+NoConn ~ 3000 1950
+NoConn ~ 3000 2250
+NoConn ~ 3000 2850
+NoConn ~ 3000 3150
 $EndSCHEMATC
