File: split56/split56.kicad_pcb (KiCad board)
At the start: 2 copper layers, 139.2 x 82 mm, 42 parts, among them J1 AudioJack4, J2 AudioJack4, J3 AudioJack4, J4 AudioJack4, SW1 SW_DIP_x02, SW10 SW_Push, SW11 SW_Push, SW12 SW_Push, SW13 SW_Push, SW14 SW_Push, SW15 SW_Push, SW16 SW_Push, SW17 SW_Push, SW18 SW_Push, SW19 SW_Push, SW2 SW_Push, SW20 SW_Push, SW21 SW_Push, SW22 SW_Push, SW23 SW_Push, SW24 SW_Push, SW25 SW_Push, SW26 SW_Push, SW27 SW_Push, SW28 SW_Push, SW29 SW_Push, SW3 SW_Push, SW4 SW_Push, SW5 SW_Push, SW6 SW_Push, SW7 SW_Push, SW8 SW_Push, SW9 SW_Push, U1 TCA9555PWR, U2 TCA9555PWR

Commit message: Add screw hole
Parts:
- added ?: Screw_Hole, library:Screw_Hole, F.Cu at (171.7, 40.4)
- added ?: Screw_Hole, library:Screw_Hole, F.Cu at (36.6, 60.3)
- added ?: Screw_Hole, library:Screw_Hole, F.Cu at (85.1, 40.4)
- added ?: Screw_Hole, library:Screw_Hole, F.Cu at (123.2, 40.4)
- added ?: Screw_Hole, library:Screw_Hole, F.Cu at (171.7, 118.4)
- added ?: Screw_Hole, library:Screw_Hole, F.Cu at (36.6, 118.4)
- added ?: Screw_Hole, library:Screw_Hole, F.Cu at (36.6, 40.4)
- added ?: Screw_Hole, library:Screw_Hole, F.Cu at (171.7, 60.3)
- added ?: Screw_Hole, library:Screw_Hole, F.Cu at (171.7, 98.4)
- added ?: Screw_Hole, library:Screw_Hole, F.Cu at (123.2, 118.4)
- added ?: Screw_Hole, library:Screw_Hole, F.Cu at (85.1, 118.4)
- added ?: Screw_Hole, library:Screw_Hole, F.Cu at (36.6, 98.4)
Routing:
- net SDA: track 162.5 -> 160.4 mm
Changed lines of the file:
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@@
     (thickness 1.6)
     (drawings 8)
-    (tracks 394)
+    (tracks 386)
     (zones 0)
-    (modules 42)
+    (modules 54)
     (nets 46)
   )
@@
       (rotate (xyz 0 0 0))
     )
+  )
+  (module library:Screw_Hole (layer F.Cu)
+    (at 171.704 40.386)
+    (fp_text reference "" (at 0 1.905) (layer F.SilkS)
+      (effects (font (size 1 1) (thickness 0.15)))
+    )
+    (fp_text value Screw_Hole (at 0 -1.905) (layer F.Fab)
+      (effects (font (size 1 1) (thickness 0.15)))
+    )
+    (pad "" np_thru_hole circle (at 0 0) (size 1.7 1.7) (drill 1.7) (layers *.Cu *.Mask))
+  )
+  (module library:Screw_Hole (layer F.Cu)
+    (at 171.704 118.364)
+    (fp_text reference "" (at 0 1.905) (layer F.SilkS)
+      (effects (font (size 1 1) (thickness 0.15)))
+    )
+    (fp_text value Screw_Hole (at 0 -1.905) (layer F.Fab)
+      (effects (font (size 1 1) (thickness 0.15)))
+    )
+    (pad "" np_thru_hole circle (at 0 0) (size 1.7 1.7) (drill 1.7) (layers *.Cu *.Mask))
+  )
+  (module library:Screw_Hole (layer F.Cu)
+    (at 36.576 118.364)
+    (fp_text reference "" (at 0 1.905) (layer F.SilkS)
+      (effects (font (size 1 1) (thickness 0.15)))
+    )
+    (fp_text value Screw_Hole (at 0 -1.905) (layer F.Fab)
+      (effects (font (size 1 1) (thickness 0.15)))
+    )
+    (pad "" np_thru_hole circle (at 0 0) (size 1.7 1.7) (drill 1.7) (layers *.Cu *.Mask))
+  )
+  (module library:Screw_Hole (layer F.Cu)
+    (at 36.576 40.386)
+    (fp_text reference "" (at 0 1.905) (layer F.SilkS)
+      (effects (font (size 1 1) (thickness 0.15)))
+    )
+    (fp_text value Screw_Hole (at 0 -1.905) (layer F.Fab)
+      (effects (font (size 1 1) (thickness 0.15)))
+    )
+    (pad "" np_thru_hole circle (at 0 0) (size 1.7 1.7) (drill 1.7) (layers *.Cu *.Mask))
+  )
+  (module library:Screw_Hole (layer F.Cu)
+    (at 171.704 60.325)
+    (fp_text reference "" (at 0 1.905) (layer F.SilkS)
+      (effects (font (size 1 1) (thickness 0.15)))
+    )
+    (fp_text value Screw_Hole (at 0 -1.905) (layer F.Fab)
+      (effects (font (size 1 1) (thickness 0.15)))
+    )
+    (pad "" np_thru_hole circle (at 0 0) (size 1.7 1.7) (drill 1.7) (layers *.Cu *.Mask))
+  )
+  (module library:Screw_Hole (layer F.Cu)
+    (at 171.704 98.425)
+    (fp_text reference "" (at 0 1.905) (layer F.SilkS)
+      (effects (font (size 1 1) (thickness 0.15)))
+    )
+    (fp_text value Screw_Hole (at 0 -1.905) (layer F.Fab)
+      (effects (font (size 1 1) (thickness 0.15)))
+    )
+    (pad "" np_thru_hole circle (at 0 0) (size 1.7 1.7) (drill 1.7) (layers *.Cu *.Mask))
+  )
+  (module library:Screw_Hole (layer F.Cu)
+    (at 123.19 118.364)
+    (fp_text reference "" (at 0 1.905) (layer F.SilkS)
+      (effects (font (size 1 1) (thickness 0.15)))
+    )
+    (fp_text value Screw_Hole (at 0 -1.905) (layer F.Fab)
+      (effects (font (size 1 1) (thickness 0.15)))
+    )
+    (pad "" np_thru_hole circle (at 0 0) (size 1.7 1.7) (drill 1.7) (layers *.Cu *.Mask))
+  )
+  (module library:Screw_Hole (layer F.Cu)
+    (at 85.09 118.364)
+    (fp_text reference "" (at 0 1.905) (layer F.SilkS)
+      (effects (font (size 1 1) (thickness 0.15)))
+    )
+    (fp_text value Screw_Hole (at 0 -1.905) (layer F.Fab)
+      (effects (font (size 1 1) (thickness 0.15)))
+    )
+    (pad "" np_thru_hole circle (at 0 0) (size 1.7 1.7) (drill 1.7) (layers *.Cu *.Mask))
+  )
+  (module library:Screw_Hole (layer F.Cu)
+    (at 36.576 98.425)
+    (fp_text reference "" (at 0 1.905) (layer F.SilkS)
+      (effects (font (size 1 1) (thickness 0.15)))
+    )
+    (fp_text value Screw_Hole (at 0 -1.905) (layer F.Fab)
+      (effects (font (size 1 1) (thickness 0.15)))
+    )
+    (pad "" np_thru_hole circle (at 0 0) (size 1.7 1.7) (drill 1.7) (layers *.Cu *.Mask))
+  )
+  (module library:Screw_Hole (layer F.Cu)
+    (at 36.576 60.325)
+    (fp_text reference "" (at 0 1.905) (layer F.SilkS)
+      (effects (font (size 1 1) (thickness 0.15)))
+    )
+    (fp_text value Screw_Hole (at 0 -1.905) (layer F.Fab)
+      (effects (font (size 1 1) (thickness 0.15)))
+    )
+    (pad "" np_thru_hole circle (at 0 0) (size 1.7 1.7) (drill 1.7) (layers *.Cu *.Mask))
+  )
+  (module library:Screw_Hole (layer F.Cu)
+    (at 85.09 40.386)
+    (fp_text reference "" (at 0 1.905) (layer F.SilkS)
+      (effects (font (size 1 1) (thickness 0.15)))
+    )
+    (fp_text value Screw_Hole (at 0 -1.905) (layer F.Fab)
+      (effects (font (size 1 1) (thickness 0.15)))
+    )
+    (pad "" np_thru_hole circle (at 0 0) (size 1.7 1.7) (drill 1.7) (layers *.Cu *.Mask))
+  )
+  (module library:Screw_Hole (layer F.Cu)
+    (at 123.19 40.386)
+    (fp_text reference "" (at 0 1.905) (layer F.SilkS)
+      (effects (font (size 1 1) (thickness 0.15)))
+    )
+    (fp_text value Screw_Hole (at 0 -1.905) (layer F.Fab)
+      (effects (font (size 1 1) (thickness 0.15)))
+    )
+    (pad "" np_thru_hole circle (at 0 0) (size 1.7 1.7) (drill 1.7) (layers *.Cu *.Mask))
   )
   (gr_arc (start 36.576 118.364) (end 34.544 118.364) (angle -90) (layer Edge.Cuts) (width 0.15))
@@
   (segment (start 111.125 103.378) (end 110.744 103.759) (width 0.25) (layer F.Cu) (net 4))
   (via (at 110.998 42.926) (size 0.8) (drill 0.4) (layers F.Cu B.Cu) (net 4))
-  (segment (start 146.615 41.6) (end 147.865 41.6) (width 0.25) (layer B.Cu) (net 4))
-  (segment (start 146.305 41.91) (end 146.615 41.6) (width 0.25) (layer B.Cu) (net 4))
-  (segment (start 131.310002 41.91) (end 146.305 41.91) (width 0.25) (layer B.Cu) (net 4))
-  (segment (start 130.075001 40.674999) (end 131.310002 41.91) (width 0.25) (layer B.Cu) (net 4))
-  (segment (start 110.998 42.926) (end 113.249001 40.674999) (width 0.25) (layer B.Cu) (net 4))
-  (segment (start 113.249001 40.674999) (end 130.075001 40.674999) (width 0.25) (layer B.Cu) (net 4))
-  (segment (start 54.175 41.91) (end 53.865 41.6) (width 0.25) (layer B.Cu) (net 4))
-  (segment (start 53.865 41.6) (end 52.615 41.6) (width 0.25) (layer B.Cu) (net 4))
-  (segment (start 108.839 40.767) (end 108.805999 40.800001) (width 0.25) (layer B.Cu) (net 4))
-  (segment (start 108.805999 40.800001) (end 72.990001 40.800001) (width 0.25) (layer B.Cu) (net 4))
-  (segment (start 58.42 41.91) (end 54.175 41.91) (width 0.25) (layer B.Cu) (net 4))
-  (segment (start 110.998 42.926) (end 108.839 40.767) (width 0.25) (layer B.Cu) (net 4))
-  (segment (start 72.990001 40.800001) (end 72.864999 40.674999) (width 0.25) (layer B.Cu) (net 4))
-  (segment (start 72.864999 40.674999) (end 59.655001 40.674999) (width 0.25) (layer B.Cu) (net 4))
-  (segment (start 59.655001 40.674999) (end 58.42 41.91) (width 0.25) (layer B.Cu) (net 4))
   (segment (start 110.998 42.926) (end 110.998 64.516) (width 0.25) (layer F.Cu) (net 4))
   (via (at 110.998 64.516) (size 0.8) (drill 0.4) (layers F.Cu B.Cu) (net 4))
@@
   (segment (start 112.776 75.858) (end 112.503001 75.585001) (width 0.25) (layer B.Cu) (net 4))
   (segment (start 112.503001 75.585001) (end 112.503001 69.704001) (width 0.25) (layer B.Cu) (net 4))
+  (segment (start 111.563685 42.926) (end 110.998 42.926) (width 0.25) (layer B.Cu) (net 4))
+  (segment (start 145.289 42.926) (end 111.563685 42.926) (width 0.25) (layer B.Cu) (net 4))
+  (segment (start 146.615 41.6) (end 145.289 42.926) (width 0.25) (layer B.Cu) (net 4))
+  (segment (start 147.865 41.6) (end 146.615 41.6) (width 0.25) (layer B.Cu) (net 4))
+  (segment (start 53.015 41.6) (end 52.615 41.6) (width 0.25) (layer B.Cu) (net 4))
+  (segment (start 54.341 42.926) (end 53.015 41.6) (width 0.25) (layer B.Cu) (net 4))
+  (segment (start 110.998 42.926) (end 54.341 42.926) (width 0.25) (layer B.Cu) (net 4))
   (segment (start 104.385 44.6) (end 104.14 44.845) (width 0.25) (layer B.Cu) (net 5))
   (segment (start 128.815 44.6) (end 104.385 44.6) (width 0.25) (layer B.Cu) (net 5))
