File: split56/split56.kicad_pcb (KiCad board)
At the start: 2 copper layers, 139.2 x 82 mm, 54 parts, among them J1 AudioJack4, J2 AudioJack4, J3 AudioJack4, J4 AudioJack4, SW1 SW_DIP_x02, SW10 SW_Push, SW11 SW_Push, SW12 SW_Push, SW13 SW_Push, SW14 SW_Push, SW15 SW_Push, SW16 SW_Push, SW17 SW_Push, SW18 SW_Push, SW19 SW_Push, SW2 SW_Push, SW20 SW_Push, SW21 SW_Push, SW22 SW_Push, SW23 SW_Push, SW24 SW_Push, SW25 SW_Push, SW26 SW_Push, SW27 SW_Push, SW28 SW_Push, SW29 SW_Push, SW3 SW_Push, SW4 SW_Push, SW5 SW_Push, SW6 SW_Push, SW7 SW_Push, SW8 SW_Push, SW9 SW_Push, U1 TCA9555PWR, U2 TCA9555PWR

Commit message: Add signature
Other:
- board text added: "by Biacco42"
Changed lines of the file:
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@@
   (general
     (thickness 1.6)
-    (drawings 8)
+    (drawings 9)
     (tracks 386)
     (zones 0)
@@
     (pad "" np_thru_hole circle (at 0 0) (size 1.7 1.7) (drill 1.7) (layers *.Cu *.Mask))
   )
+  (gr_text "by Biacco42" (at 161.544 117.602) (layer F.SilkS)
+    (effects (font (size 1.5 1.5) (thickness 0.3)))
+  )
   (gr_arc (start 36.576 118.364) (end 34.544 118.364) (angle -90) (layer Edge.Cuts) (width 0.15))
